Commit message: Experience-driven Predictive Control full stack formulation implemented

File: Tools/sitl_gazebo/models/rotors_description/urdf/component_snippets.xacro (robot description, xacro)
@@ -110,9 +110,9 @@
       <plugin name="controller_interface" filename="librotors_gazebo_controller_interface.so">
         <robotNamespace>${namespace}</robotNamespace>
-        <commandAttitudeThrustSubTopic>/command/attitude</commandAttitudeThrustSubTopic>
-        <commandRateThrustSubTopic>/command/rate</commandRateThrustSubTopic>
-        <commandMotorSpeedSubTopic>/command/motor_speed</commandMotorSpeedSubTopic>
-        <imuSubTopic>/${imu_sub_topic}</imuSubTopic>
-        <motorSpeedCommandPubTopic>/gazebo/command/motor_speed</motorSpeedCommandPubTopic>
+        <commandAttitudeThrustSubTopic>command/attitude</commandAttitudeThrustSubTopic>
+        <commandRateThrustSubTopic>command/rate</commandRateThrustSubTopic>
+        <commandMotorSpeedSubTopic>command/motor_speed</commandMotorSpeedSubTopic>
+        <imuSubTopic>${imu_sub_topic}</imuSubTopic>
+        <motorSpeedCommandPubTopic>gazebo/command/motor_speed</motorSpeedCommandPubTopic>
       </plugin>
     </gazebo>
@@ -124,5 +124,5 @@
         <robotNamespace>${namespace}</robotNamespace>
         <imuSubTopic>${imu_sub_topic}</imuSubTopic>
-        <motorSpeedCommandPubTopic>/gazebo/command/motor_speed</motorSpeedCommandPubTopic>
+        <motorSpeedCommandPubTopic>gazebo/command/motor_speed</motorSpeedCommandPubTopic>
       </plugin>
     </gazebo>
@@ -419,5 +419,5 @@
       imu_suffix=""
       parent_link="${namespace}/vi_sensor_link"
-      imu_topic="/imu"
+      imu_topic="imu"
       mass_imu_sensor="0.015"
       gyroscope_noise_density="0.0003394"

File: Tools/sitl_gazebo/models/rotors_description/urdf/iris.xacro (robot description, xacro)
@@ -4,5 +4,5 @@
   <xacro:property name="namespace" value="iris" />
   <xacro:property name="rotor_velocity_slowdown_sim" value="10" />
-  <xacro:property name="mesh_file" value="iris.stl" />
+  <xacro:property name="mesh_file" value="iris.dae" />
   <xacro:property name="mesh_scale" value="1 1 1"/>
   <xacro:property name="mesh_scale_prop" value="1 1 1"/>
@@ -16,14 +16,14 @@
   <xacro:property name="arm_length_back_y" value="0.2" /> <!-- [m] -->
   <xacro:property name="rotor_offset_top" value="0.023" /> <!-- [m] -->
-  <xacro:property name="radius_rotor" value="0.128" /> <!-- [m] -->
+  <xacro:property name="radius_rotor" value="0.1" /> <!-- [m] -->
   <xacro:property name="motor_constant" value="8.54858e-06" /> <!-- [kg.m/s^2] -->
-  <xacro:property name="moment_constant" value="0.06" /> <!-- [m] -->
+  <xacro:property name="moment_constant" value="0.16" /> <!-- [m] -->
   <xacro:property name="time_constant_up" value="0.0125" /> <!-- [s] -->
   <xacro:property name="time_constant_down" value="0.025" /> <!-- [s] -->
-  <xacro:property name="max_rot_velocity" value="1100" /> <!-- [rad/s] -->
+  <xacro:property name="max_rot_velocity" value="838" /> <!-- [rad/s] -->
   <xacro:property name="sin30" value="0.5" />
   <xacro:property name="cos30" value="0.866025403784" />
   <xacro:property name="sqrt2" value="1.4142135623730951" />
-  <xacro:property name="rotor_drag_coefficient" value="8.06428e-04" />
+  <xacro:property name="rotor_drag_coefficient" value="8.06428e-05" />
   <xacro:property name="rolling_moment_coefficient" value="0.000001" />
   <xacro:property name="color" value="DarkGrey" />

File: Tools/sitl_gazebo/models/rotors_description/urdf/iris_base.xacro (robot description, xacro)
@@ -8,5 +8,5 @@
   <xacro:mavlink_interface_macro
     namespace="${namespace}"
-    imu_sub_topic="/imu"
+    imu_sub_topic="imu"
     >
   </xacro:mavlink_interface_macro>
@@ -17,5 +17,5 @@
     imu_suffix=""
     parent_link="base_link"
-    imu_topic="/imu"
+    imu_topic="imu"
     mass_imu_sensor="0.015"
     gyroscope_noise_density="0.0003394"

File: Tools/sitl_gazebo/models/rotors_description/urdf/multirotor_base.xacro (robot description, xacro)
@@ -57,18 +57,5 @@
     <gazebo reference="base_link">
       <material>Gazebo/${color}</material>
-      <collision name='base_link_inertia_collision'>
-        <surface>
-          <contact>
-            <ode>
-              <min_depth>0.001</min_depth>
-              <max_vel>0.0</max_vel>
-            </ode>
-          </contact>
-          <friction>
-            <ode/>
-          </friction>
-        </surface>
-      </collision>
-   </gazebo>
+    </gazebo>
   </xacro:macro>
   <!-- Rotor joint and link -->
@@ -117,9 +104,9 @@
         <motorConstant>${motor_constant}</motorConstant>
         <momentConstant>${moment_constant}</momentConstant>
-        <commandSubTopic>/gazebo/command/motor_speed</commandSubTopic>
+        <commandSubTopic>gazebo/command/motor_speed</commandSubTopic>
         <motorNumber>${motor_number}</motorNumber>
         <rotorDragCoefficient>${rotor_drag_coefficient}</rotorDragCoefficient>
         <rollingMomentCoefficient>${rolling_moment_coefficient}</rollingMomentCoefficient>
-        <motorSpeedPubTopic>/motor_speed/${motor_number}</motorSpeedPubTopic>
+        <motorSpeedPubTopic>motor_speed/${motor_number}</motorSpeedPubTopic>
         <rotorVelocitySlowdownSim>${rotor_velocity_slowdown_sim}</rotorVelocitySlowdownSim>
       </plugin>
